File: kicad/hwpboard.sch (KiCad schematic (older format))
At the start: 5 parts, among them J1 Barrel_Jack_Switch, J2 Conn_01x01, J3 Conn_01x01, J4 Conn_01x01, J5 Conn_01x01

Commit message: Schematic almost done.
Parts:
- added C1, C2, C? (x2): 100n, symbol Device:C
- added LCD1602: RC1602A, HWP:WC1602A, symbol Display_Character:RC1602A
- added MoistureSensor1: Conn_01x05_Male, HWP:WC1602A, symbol Connector:Conn_01x05_Male
- added NUCBRD1: NUCLEO64, HWP:ST_Morpho_Connector_STLink, symbol HWP:NUCLEO64
- added PushButton1: SW_Push, symbol Switch:SW_Push
- added R1: 10k, Resistor_SMD:R_0805_2012Metric_Pad1.15x1.40mm_HandSolder, symbol Device:R
- added R2: 6k, Resistor_SMD:R_0805_2012Metric_Pad1.15x1.40mm_HandSolder, symbol Device:R
- added R3, R4, R? (x2): 50k, symbol Device:R
- added RotaryEncoder1: Rotary_Encoder_Switch, Rotary_Encoder:RotaryEncoder_Alps_EC11E-Switch_Vertical_H20mm, symbol Device:Rotary_Encoder_Switch
- added U1: AD8603, Package_TO_SOT_SMD:TSOT-23-5, symbol Amplifier_Operational:AD8603
Connections:
- net labels added: +3.3V, 3V3, ADC, DAC0, DAC1, E, GNDA, LCD_out, PWM, RS, brightness, btn0, btn1, contrast, d0, d1, d2, d3, d4, d5, d6, d7, humid_out, rotary0, rotary1, temp_out
- wire segments 4 -> 97
- no-connect marks 5 -> 47
