File: kicad/hwpboard.sch (KiCad schematic (older format))
At the start: 24 parts, among them J1 Barrel_Jack_Switch, J2 Conn_01x01, J3 Conn_01x01, J4 Conn_01x01, J5 Conn_01x01, U1 AD8603

Commit message: layout_all_routed_and_drc_ok_v_1.0
Parts:
- PushButton1: footprint (none) -> HWP:SW_PUSH_6mm
- RotaryEncoder1: footprint Rotary_Encoder:RotaryEncoder_Alps_EC11E-Switch_Vertical_H20mm -> HWP:RotaryEncoder_Alps_EC12E-Switch_Vertical_H20mm_CircularMountingHoles
Connections:
- net labels removed: ADC, LCD_out, contrast
Changed lines of the file:
@@
 F 0 "RotaryEncoder1" H 9900 3617 50  0000 C CNN
 F 1 "Rotary_Encoder_Switch" H 9900 3526 50  0000 C CNN
-F 2 "Rotary_Encoder:RotaryEncoder_Alps_EC11E-Switch_Vertical_H20mm" H 9750 3410 50  0001 C CNN
+F 2 "HWP:RotaryEncoder_Alps_EC12E-Switch_Vertical_H20mm_CircularMountingHoles" H 9750 3410 50  0001 C CNN
 F 3 "~" H 9900 3510 50  0001 C CNN
 	1    9900 3250
@@
 $EndComp
 Wire Wire Line
-	3900 3850 3350 3850
-Wire Wire Line
-	3900 3950 3350 3950
-Text Label 3350 3850 0    50   ~ 0
-ADC
-Text Label 3350 3950 0    50   ~ 0
-ADC
-Wire Wire Line
 	6100 2650 6650 2650
 Wire Wire Line
@@
 Wire Wire Line
 	9200 6050 9200 6250
-Text Label 9200 6050 0    50   ~ 0
-brightness
 Wire Wire Line
 	9100 5550 9300 5550
-Text Label 9550 5550 0    50   ~ 0
-contrast
 Wire Wire Line
 	8300 5350 8250 5350
@@
 	7650 7450 7650 7600
 Wire Wire Line
-	7400 7150 7900 7150
-Wire Wire Line
-	7400 7250 7900 7250
-Wire Wire Line
 	7400 7350 7900 7350
-Text Label 6650 3050 0    50   ~ 0
-LCD_out
-Text Label 6650 3150 0    50   ~ 0
-LCD_out
-Text Label 6650 3250 0    50   ~ 0
-LCD_out
-Text Label 6650 3350 0    50   ~ 0
-LCD_out
-Text Label 6650 3450 0    50   ~ 0
-LCD_out
-Text Label 6650 3550 0    50   ~ 0
-LCD_out
-Text Label 3400 4450 0    50   ~ 0
-LCD_out
-Text Label 3400 4550 0    50   ~ 0
-LCD_out
-Text Label 3400 4650 0    50   ~ 0
-LCD_out
-Text Label 3400 4750 0    50   ~ 0
-LCD_out
 Wire Wire Line
 	6100 5350 6700 5350
@@
 F 0 "PushButton1" H 9850 2485 50  0000 C CNN
 F 1 "SW_Push" H 9850 2394 50  0000 C CNN
-F 2 "" H 9850 2400 50  0001 C CNN
+F 2 "HWP:SW_PUSH_6mm" H 9850 2400 50  0001 C CNN
 F 3 "" H 9850 2400 50  0001 C CNN
 	1    9850 2200
@@
 Text GLabel 9300 5550 2    50   Input ~ 0
 DAC0
-Text Label 6950 2650 0    50   ~ 0
-contrast
-Text Label 6950 2750 0    50   ~ 0
-brightness
-Text Label 5550 7100 0    50   ~ 0
-brightness
 Wire Wire Line
 	5550 7400 6100 7400
@@
 	10350 5750 10350 5950
 Connection ~ 10350 5950
+Wire Wire Line
+	3350 3850 3900 3850
+Wire Wire Line
+	3900 3950 3350 3950
+Wire Wire Line
+	7900 7150 7400 7150
+Wire Wire Line
+	7400 7250 7900 7250
 $EndSCHEMATC

Commit message: layout_all_routed_and_drc_ok_beta_2.0
Parts:
- removed C1, C2, C3, C4, C6: 100n, Capacitor_SMD:C_0805_2012Metric_Pad1.15x1.40mm_HandSolder, symbol Device:C
- removed R1: 10k, Resistor_SMD:R_0805_2012Metric_Pad1.15x1.40mm_HandSolder, symbol Device:R
- removed R2: 6.2k, Resistor_SMD:R_0805_2012Metric_Pad1.15x1.40mm_HandSolder, symbol Device:R
- removed R3, R4, R5, R6: 50k, Resistor_SMD:R_0805_2012Metric_Pad1.15x1.40mm_HandSolder, symbol Device:R
- removed U1: AD8603, Package_TO_SOT_SMD:TSOT-23-5, symbol Amplifier_Operational:AD8603
- added C3: 100u, HWP:CP_Radial_D7.5mm_P2.50mm, symbol Device:CP
- added Dz1: ZEN056V115A24LS, Diode_SMD:Littelfuse_PolyZen-LS, symbol Power_Protection:ZEN056V115A24LS
- added Q1: BSS138, Package_TO_SOT_SMD:SOT-23, symbol Transistor_FET:BSS138
- C1: renamed from C5; footprint Capacitor_SMD:C_0805_2012Metric_Pad1.15x1.40mm_HandSolder -> HWP:C_0805_2012Metric_Pad1.15x1.40mm_HandSolder
- C2: renamed from C7; footprint Capacitor_SMD:C_0805_2012Metric_Pad1.15x1.40mm_HandSolder -> HWP:C_0805_2012Metric_Pad1.15x1.40mm_HandSolder
- LCD1: renamed from LCD1602; footprint HWP:WC1602A -> HWP:WC1602A_no_mount
Connections:
- net labels added: PWM_LCD, PWM_sensor, Sensor_enable
- net labels removed: 3V3, DAC1, GNDA, PWM
- wire segments 110 -> 89
- no-connect marks 47 -> 46
Other:
- note added: "Control buttons"
- note added: "LCD module"
- note added: "PWM driver for the LCD backlight"
- note added: "Sensor connector"
- note removed: "need real rail-to-rail opamp for full brightness\n"
