File: kicad/_saved_hwpboard.sch (KiCad schematic (older format))
At the start: 24 parts, among them J1 Barrel_Jack_Switch, J2 Conn_01x01, J3 Conn_01x01, J4 Conn_01x01, J5 Conn_01x01, U1 AD8603

Commit message: schematic v1.0 ready
Parts:
- PushButton1: footprint (none) -> HWP:SW_PUSH_6mm
- RotaryEncoder1: footprint Rotary_Encoder:RotaryEncoder_Alps_EC11E-Switch_Vertical_H20mm -> HWP:RotaryEncoder_Alps_EC12E-Switch_Vertical_H20mm_CircularMountingHoles
Changed lines of the file:
@@
 F 0 "RotaryEncoder1" H 9900 3617 50  0000 C CNN
 F 1 "Rotary_Encoder_Switch" H 9900 3526 50  0000 C CNN
-F 2 "Rotary_Encoder:RotaryEncoder_Alps_EC11E-Switch_Vertical_H20mm" H 9750 3410 50  0001 C CNN
+F 2 "HWP:RotaryEncoder_Alps_EC12E-Switch_Vertical_H20mm_CircularMountingHoles" H 9750 3410 50  0001 C CNN
 F 3 "~" H 9900 3510 50  0001 C CNN
 	1    9900 3250
@@
 F 0 "PushButton1" H 9850 2485 50  0000 C CNN
 F 1 "SW_Push" H 9850 2394 50  0000 C CNN
-F 2 "" H 9850 2400 50  0001 C CNN
+F 2 "HWP:SW_PUSH_6mm" H 9850 2400 50  0001 C CNN
 F 3 "" H 9850 2400 50  0001 C CNN
 	1    9850 2200
