File: kicad/_saved_hwpboard.sch (KiCad schematic (older format))
At the start: 17 parts, among them J1 Barrel_Jack_Switch, J2 Conn_01x01, J3 Conn_01x01, J4 Conn_01x01, J5 Conn_01x01, Q1 BSS138

Commit message: Board finished and checked
Parts:
- Rm1: value 10000 -> 100k
Changed lines of the file:
@@
 P 4350 7600
 F 0 "Rm1" H 4420 7646 50  0000 L CNN
-F 1 "10000" H 4420 7555 50  0000 L CNN
+F 1 "100k" H 4420 7555 50  0000 L CNN
 F 2 "HWP:R_0805_2012Metric_Pad1.15x1.40mm_HandSolder" V 4280 7600 50  0001 C CNN
 F 3 "~" H 4350 7600 50  0001 C CNN
