File: kicad/hwpboard.kicad_pcb (KiCad board)
At the start: 2 copper layers, 100 x 80 mm, 17 parts, among them J1 Barrel_Jack_Switch, J2 Conn_01x01, J3 Conn_01x01, J4 Conn_01x01, J5 Conn_01x01, Q1 BSS138

Commit message: some edits
Parts:
- Rm1: value 10000 -> 100k
- moved Q1 0.96 mm to (125.7, 90.7), turned to 90 degrees
Routing:
- net Net-(Q1-Pad1): track 11.0 -> 5.18 mm
- net DAC0: track 120.1 -> 121.8 mm
Changed lines of the file:
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@@
     (thickness 1.6)
     (drawings 15)
-    (tracks 175)
+    (tracks 171)
     (zones 0)
     (modules 17)
@@
   )
   (setup
-    (last_trace_width 0.6096)
+    (last_trace_width 0.4064)
     (user_trace_width 0.3048)
     (user_trace_width 0.4064)
     (user_trace_width 0.6096)
     (trace_clearance 0.2)
-    (zone_clearance 0.508)
+    (zone_clearance 0.708)
     (zone_45_only no)
     (trace_min 0.2)
@@
     (visible_elements 7FFFFFFF)
     (pcbplotparams
-      (layerselection 0x011c0_ffffffff)
+      (layerselection 0x010c0_ffffffff)
       (usegerberextensions false)
       (usegerberattributes false)
@@
   )
   (module Package_TO_SOT_SMD:SOT-23 (layer F.Cu)
-    (at 124.822 91.152)
+    (at 125.65 90.66 90)
     (descr "SOT-23, Standard")
     (tags SOT-23)
     (attr smd)
-    (fp_text reference Q1 (at 0 -2.5) (layer F.SilkS)
-      (effects (font (size 1 1) (thickness 0.15)))
-    )
-    (fp_text value BSS138 (at 0 2.5) (layer F.Fab)
-      (effects (font (size 1 1) (thickness 0.15)))
-    )
-    (fp_text user %R (at 0 0 -270) (layer F.Fab)
+    (fp_text reference Q1 (at 0 -2.5 90) (layer F.SilkS)
+      (effects (font (size 1 1) (thickness 0.15)))
+    )
+    (fp_text value BSS138 (at 0 2.5 90) (layer F.Fab)
+      (effects (font (size 1 1) (thickness 0.15)))
+    )
+    (fp_text user %R (at 0 0 -180) (layer F.Fab)
       (effects (font (size 0.5 0.5) (thickness 0.075)))
     )
@@
     (fp_line (start 0.76 -1.58) (end -1.4 -1.58) (layer F.SilkS) (width 0.12))
     (fp_line (start 0.76 1.58) (end -0.7 1.58) (layer F.SilkS) (width 0.12))
-    (pad 1 smd rect (at -1 -0.95) (size 0.9 0.8) (layers F.Cu F.Paste F.Mask)
+    (pad 1 smd rect (at -1 -0.95 90) (size 0.9 0.8) (layers F.Cu F.Paste F.Mask)
       (net 25 "Net-(Q1-Pad1)"))
-    (pad 2 smd rect (at -1 0.95) (size 0.9 0.8) (layers F.Cu F.Paste F.Mask)
-      (net 1 GND))
-    (pad 3 smd rect (at 1 0) (size 0.9 0.8) (layers F.Cu F.Paste F.Mask)
+    (pad 2 smd rect (at -1 0.95 90) (size 0.9 0.8) (layers F.Cu F.Paste F.Mask)
+      (net 1 GND))
+    (pad 3 smd rect (at 1 0 90) (size 0.9 0.8) (layers F.Cu F.Paste F.Mask)
       (net 5 brightness))
     (model ${KISYS3DMOD}/Package_TO_SOT_SMD.3dshapes/SOT-23.wrl
@@
       (effects (font (size 1 1) (thickness 0.15)))
     )
-    (fp_text value 10000 (at 0 1.65 180) (layer F.Fab)
+    (fp_text value 100k (at 0 1.65 180) (layer F.Fab)
       (effects (font (size 1 1) (thickness 0.15)))
     )
@@
     )
   )
+  (gr_text GND (at 110.09 78.325) (layer F.Cu)
+    (effects (font (size 1 1) (thickness 0.2) italic) (justify left))
+  )
   (gr_text - (at 117.71 49.75) (layer F.Cu)
     (effects (font (size 1.5 1.5) (thickness 0.2)) (justify left))
@@
   )
   (gr_text "En  " (at 110.09 88.485) (layer F.Cu)
-    (effects (font (size 1.5 1.5) (thickness 0.2) italic) (justify left))
+    (effects (font (size 1 1) (thickness 0.2) italic) (justify left))
   )
   (gr_text Hum (at 110.09 85.945) (layer F.Cu)
-    (effects (font (size 1.5 1.5) (thickness 0.2) italic) (justify left))
+    (effects (font (size 1 1) (thickness 0.2) italic) (justify left))
   )
   (gr_text Tmp (at 110.09 83.405) (layer F.Cu)
-    (effects (font (size 1.5 1.5) (thickness 0.2) italic) (justify left))
+    (effects (font (size 1 1) (thickness 0.2) italic) (justify left))
   )
   (gr_text PWM (at 110.09 80.865) (layer F.Cu)
-    (effects (font (size 1.5 1.5) (thickness 0.2) italic) (justify left))
-  )
-  (gr_text GND (at 110.09 78.325) (layer F.Cu)
-    (effects (font (size 1.5 1.5) (thickness 0.2) italic) (justify left))
+    (effects (font (size 1 1) (thickness 0.2) italic) (justify left))
   )
   (dimension 80.01 (width 0.3) (layer Dwgs.User)
@@
   (gr_line (start 208.81 42.14) (end 208.81 122.14) (layer Edge.Cuts) (width 0.15))
   (gr_line (start 108.81 42.14) (end 208.81 42.14) (layer Edge.Cuts) (width 0.15))
-  (via (at 122.79 94.2) (size 1) (drill 0.4) (layers F.Cu B.Cu) (net 1))
+  (via (at 127.87 94.2) (size 1) (drill 0.4) (layers F.Cu B.Cu) (net 1))
   (segment (start 160.89 53.56) (end 160.89 77.055) (width 0.6096) (layer B.Cu) (net 2))
   (segment (start 160.89 77.055) (end 158.985 78.96) (width 0.6096) (layer B.Cu) (net 2))
@@
   (segment (start 130.41 78.96) (end 133.34 78.96) (width 0.6096) (layer F.Cu) (net 2))
   (segment (start 130.41 111.98) (end 126.6 111.98) (width 0.6096) (layer F.Cu) (net 2))
-  (segment (start 177.4 52.29) (end 178.67 53.56) (width 0.3048) (layer F.Cu) (net 3))
-  (segment (start 142.475 49.115) (end 176.004554 49.115) (width 0.3048) (layer F.Cu) (net 3))
-  (segment (start 141.84 73.88) (end 141.84 49.75) (width 0.3048) (layer F.Cu) (net 3))
-  (segment (start 141.84 49.75) (end 142.475 49.115) (width 0.3048) (layer F.Cu) (net 3))
-  (segment (start 125.965 109.44) (end 124.949 108.424) (width 0.3048) (layer F.Cu) (net 3))
-  (segment (start 130.41 109.44) (end 125.965 109.44) (width 0.3048) (layer F.Cu) (net 3))
-  (segment (start 176.004554 49.115) (end 177.4 50.510446) (width 0.3048) (layer F.Cu) (net 3))
-  (segment (start 124.949 76.166) (end 126.6 74.515) (width 0.3048) (layer F.Cu) (net 3))
-  (segment (start 177.4 50.510446) (end 177.4 52.29) (width 0.3048) (layer F.Cu) (net 3))
-  (segment (start 124.949 108.424) (end 124.949 76.166) (width 0.3048) (layer F.Cu) (net 3))
-  (segment (start 126.6 74.515) (end 141.205 74.515) (width 0.3048) (layer F.Cu) (net 3))
-  (segment (start 141.205 74.515) (end 141.84 73.88) (width 0.3048) (layer F.Cu) (net 3))
+  (segment (start 178.67 78.96) (end 178.67 78.425554) (width 0.3048) (layer B.Cu) (net 3))
+  (segment (start 138.03 115.79) (end 138.03 84.04) (width 0.3048) (layer B.Cu) (net 3))
+  (segment (start 178.67 78.425554) (end 178.67 53.56) (width 0.3048) (layer B.Cu) (net 3))
+  (segment (start 130.41 109.44) (end 127.87 109.44) (width 0.3048) (layer B.Cu) (net 3))
+  (segment (start 176.13 81.5) (end 178.67 78.96) (width 0.3048) (layer B.Cu) (net 3))
+  (segment (start 140.57 81.5) (end 176.13 81.5) (width 0.3048) (layer B.Cu) (net 3))
+  (segment (start 138.03 84.04) (end 140.57 81.5) (width 0.3048) (layer B.Cu) (net 3))
+  (segment (start 127.87 109.44) (end 126.6 110.71) (width 0.3048) (layer B.Cu) (net 3))
+  (segment (start 126.6 115.79) (end 127.87 117.06) (width 0.3048) (layer B.Cu) (net 3))
+  (segment (start 126.6 110.71) (end 126.6 115.79) (width 0.3048) (layer B.Cu) (net 3))
+  (segment (start 127.87 117.06) (end 136.76 117.06) (width 0.3048) (layer B.Cu) (net 3))
+  (segment (start 136.76 117.06) (end 138.03 115.79) (width 0.3048) (layer B.Cu) (net 3))
   (segment (start 140.57 111.98) (end 140.57 103.09) (width 0.3048) (layer F.Cu) (net 4))
   (segment (start 139.3 101.82) (end 130.41 101.82) (width 0.3048) (layer F.Cu) (net 4))
   (segment (start 140.57 103.09) (end 139.3 101.82) (width 0.3048) (layer F.Cu) (net 4))
-  (segment (start 126.584 90.39) (end 125.822 91.152) (width 0.6096) (layer F.Cu) (net 5))
-  (segment (start 126.6 90.39) (end 126.584 90.39) (width 0.6096) (layer F.Cu) (net 5))
-  (segment (start 130.41 76.42) (end 130.01 76.42) (width 0.6096) (layer F.Cu) (net 5))
-  (segment (start 126.6 90.39) (end 127.235 89.755) (width 0.6096) (layer F.Cu) (net 5))
-  (segment (start 127.235 89.755) (end 127.235 79.195) (width 0.6096) (layer F.Cu) (net 5))
-  (segment (start 130.01 76.42) (end 127.235 79.195) (width 0.6096) (layer F.Cu) (net 5))
+  (segment (start 126.6 77.69) (end 127.87 76.42) (width 0.6096) (layer F.Cu) (net 5))
+  (segment (start 127.87 76.42) (end 130.41 76.42) (width 0.6096) (layer F.Cu) (net 5))
+  (segment (start 126.6 87.6504) (end 126.6 77.69) (width 0.6096) (layer F.Cu) (net 5))
+  (segment (start 125.65 89.66) (end 125.65 88.6004) (width 0.6096) (layer F.Cu) (net 5))
+  (segment (start 125.65 88.6004) (end 126.6 87.6504) (width 0.6096) (layer F.Cu) (net 5))
   (segment (start 188.18259 51.66741) (end 186.29 53.56) (width 0.3048) (layer F.Cu) (net 6))
   (segment (start 139.3 49.115) (end 139.935 48.48) (width 0.3048) (layer F.Cu) (net 6))
@@
   (segment (start 143.11 99.28) (end 141.84 98.01) (width 0.3048) (layer F.Cu) (net 24))
   (segment (start 125.965 96.105) (end 125.965 100.55) (width 0.3048) (layer F.Cu) (net 24))
-  (segment (start 122.978 90.202) (end 123.822 90.202) (width 0.3048) (layer F.Cu) (net 25))
-  (segment (start 121.708 90.202) (end 122.978 90.202) (width 0.3048) (layer F.Cu) (net 25))
-  (segment (start 120.885 91.025) (end 121.708 90.202) (width 0.3048) (layer F.Cu) (net 25))
-  (segment (start 123.915 96.105) (end 121.52 96.105) (width 0.3048) (layer F.Cu) (net 25))
-  (segment (start 120.885 95.47) (end 120.885 91.025) (width 0.3048) (layer F.Cu) (net 25))
-  (segment (start 121.52 96.105) (end 120.885 95.47) (width 0.3048) (layer F.Cu) (net 25))
+  (segment (start 123.9952 91.66) (end 124.7 91.66) (width 0.3048) (layer F.Cu) (net 25))
+  (segment (start 123.915 91.7402) (end 123.9952 91.66) (width 0.3048) (layer F.Cu) (net 25))
+  (segment (start 123.915 96.105) (end 123.915 91.7402) (width 0.3048) (layer F.Cu) (net 25))
   (zone (net 1) (net_name GND) (layer B.Cu) (hatch none 0.508)
     (connect_pads (clearance 0.508))
